File: hardware/8085.brd (EAGLE design)
At the start: 167.9 x 122.5 mm, 49 parts, among them IC10 74HCT00N, IC11 74HCT245DW, IC2 74AC573N, IC3 ATF16V8BP3, IC4 74AC00D, IC5 74HCT245DW, IC6 74AC273N, IC7 74HCT139N, IC8 7404N, IC9 74HCT138N

Commit message: PCB design upadted
Parts:
- C5: device rcl:C050-024X044 -> rcl:C0603
- R1: device rcl:0204/7 -> rcl:0204/5
- R10: device rcl:R0603 -> rcl:0207/10
- R8: device rcl:0204/7 -> rcl:0207/10
- moved C5 79.2 mm to (45.3, 38.0), flipped to the bottom
- moved C16 50.4 mm to (10.9, 31.4), turned to 0 degrees
- moved R10 15.3 mm to (19.1, 24.8), flipped to the top, turned to 180 degrees
- moved R8 15.3 mm to (17.8, 27.3)
- moved JP1 14.7 mm to (8.26, 51.4), turned to 180 degrees
- moved R1 7.41 mm to (9.53, 48.6)
- moved R11 6.27 mm to (45.8, 26.0), turned to 0 degrees
- moved C23 4.45 mm to (46.7, 111.8)
- moved C22 2.54 mm to (18.2, 109.9)
- moved IC1 2.54 mm to (24.1, 60.3)
- moved IC4 2.54 mm to (24.1, 106.0)
- moved C11 2.54 mm to (16.5, 33.0)
- moved C18 2.54 mm to (19.1, 100.0)
- moved C4 2.54 mm to (9.53, 46.4)
- moved D1 2.54 mm to (8.26, 43.8)
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Connections:
- net CF_D0: now also IC11.16; no longer IC11.18
- net CF_D2: now also IC11.18; no longer IC11.16
- net D0: now also IC11.4; no longer IC11.2
- net D2: now also IC11.2; no longer IC11.4
- net IO_M: now also IC3.6; no longer IC3.3
- net LOCAL_IO_CS: now also IC3.7; no longer IC3.6
Routing:
- net RD: track 5.40 -> 107.0 mm, vias 0 -> 2
- net IO_M: track 9.89 -> 101.4 mm, vias 0 -> 2
- net A2: track 124.3 -> 180.1 mm, vias 0 -> 2
- net A1: track 132.7 -> 185.3 mm, vias 2 -> 4
- net VCC: track 568.0 -> 616.8 mm, vias 6 -> 10
- net A0: track 153.0 -> 198.9 mm, vias 4 -> 6
- net CF_D2: track 0.00 -> 29.0 mm
- net CF_D1: track 0.00 -> 29.0 mm
- net CF_D0: track 0.00 -> 29.0 mm
- net N$11: track 0.00 -> 25.9 mm
- net N$13: track 0.00 -> 18.7 mm
- net GND: track 118.0 -> 129.9 mm, vias 10 -> 12
- net A4: track 178.9 -> 187.8 mm
- net INT: track 136.5 -> 144.7 mm
- net N$29: track 3.23 -> 11.2 mm
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
Commit message: Minor PCB updates
Parts:
- added C7: 100n, rcl:C0603
- added C8: 22p, rcl:C0603
- added JP3: (no value), pinhead:1X02
- R11, R7: device rcl:R0603 -> rcl:0204/7
- moved R7 12.0 mm to (56.5, 30.1), turned to 180 degrees
- moved R11 10.8 mm to (56.5, 27.6), turned to 180 degrees
Connections:
- net GND: now also C7.2, C8.1, JP3.2
- net N$2: now also C8.2
- net VCC: now also C7.1, JP3.1
Routing:
- net VCC: track 616.8 -> 639.1 mm
- net N$12: track 3.52 -> 11.7 mm
- net N$29: track 11.2 -> 6.57 mm
- net N$2: track 4.92 -> 6.61 mm
- net GND: track 129.9 -> 131.1 mm
Changed lines of the file:
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@@
 <attribute name="OC_FARNELL" value="unknown" x="44.7675" y="2.54" size="1.778" layer="28" rot="MR180" display="off"/>
 </element>
-<element name="R7" library="rcl" package="R0603" value="" x="45.8343" y="24.5364" rot="MR0"/>
+<element name="R7" library="rcl" package="0204/7" value="" x="56.515" y="30.0736" rot="MR180"/>
 <element name="R8" library="rcl" package="0207/10" value="" x="17.78" y="27.305" rot="R180"/>
 <element name="R10" library="rcl" package="0207/10" value="" x="19.05" y="24.765" rot="R180"/>
-<element name="R11" library="rcl" package="R0603" value="" x="45.8343" y="26.035" rot="MR0"/>
+<element name="R11" library="rcl" package="0204/7" value="" x="56.515" y="27.6225" rot="MR180"/>
 <element name="RN1" library="resistor-sil" package="SIL5" value="" x="35.56" y="53.975" rot="R270">
 <attribute name="OC_NEWARK" value="unknown" x="35.56" y="53.975" size="1.778" layer="27" rot="R270" display="off"/>
@@
 <element name="R4" library="rcl" package="0204/7" value="" x="8.255" y="46.355" rot="R180"/>
 <element name="C4" library="rcl" package="C0603" value="" x="9.525" y="46.355" rot="MR0"/>
+<element name="JP3" library="pinhead" package="1X02" value="" x="23.1775" y="115.57" rot="R90"/>
+<element name="C7" library="rcl" package="C0603" value="100n" x="44.7675" y="25.6159" rot="MR90"/>
+<element name="C8" library="rcl" package="C0603" value="22p" x="38.735" y="39.878" rot="MR0"/>
 </elements>
 <signals>
@@
 <contactref element="R11" pad="2"/>
 <contactref element="R10" pad="2"/>
-<wire x1="45.085" y1="21.32" x2="45.085" y2="24.5364" width="0.4064" layer="16"/>
-<wire x1="44.45" y1="21.32" x2="44.45" y2="24.892" width="0.4064" layer="16"/>
-<wire x1="44.45" y1="24.892" x2="45.085" y2="24.892" width="0.4064" layer="16"/>
 <contactref element="D1" pad="C"/>
 <contactref element="R4" pad="2"/>
@@
 <via x="39.0525" y="114.3" extent="1-16" drill="0.6" diameter="1.778" shape="octagon"/>
 <wire x1="39.0525" y1="60.325" x2="39.0525" y2="114.3" width="0.6096" layer="1"/>
-<wire x1="44.9843" y1="24.5364" x2="45.085" y2="24.5364" width="0.4064" layer="16"/>
-<wire x1="45.085" y1="24.5364" x2="45.085" y2="24.892" width="0.4064" layer="16"/>
 <wire x1="4.445" y1="104.775" x2="13.97" y2="114.3" width="1.27" layer="16"/>
-<wire x1="44.9843" y1="24.5364" x2="44.9843" y2="24.6643" width="0.4064" layer="16"/>
-<wire x1="44.9843" y1="24.5364" x2="44.9843" y2="24.8675" width="0.4064" layer="16"/>
 <wire x1="43.18" y1="37.1983" x2="45.085" y2="37.1983" width="0.6096" layer="16"/>
 <wire x1="45.085" y1="37.1983" x2="47.625" y2="37.1983" width="0.6096" layer="16"/>
@@
 <wire x1="43.18" y1="39.1033" x2="43.18" y2="58.7883" width="0.6096" layer="1"/>
 <via x="43.18" y="37.1983" extent="1-16" drill="0.6" diameter="1.4224" shape="octagon"/>
-<via x="43.18" y="24.5364" extent="1-16" drill="0.6" diameter="1.4224" shape="octagon"/>
-<wire x1="43.18" y1="24.5364" x2="43.18" y2="37.1983" width="0.6096" layer="1"/>
-<wire x1="43.18" y1="24.5364" x2="44.9843" y2="24.5364" width="0.6096" layer="16"/>
-<wire x1="44.9843" y1="26.035" x2="44.9843" y2="24.5364" width="0.6096" layer="16"/>
+<via x="43.18" y="24.7659" extent="1-16" drill="0.6" diameter="1.4224" shape="octagon"/>
+<wire x1="43.18" y1="24.7659" x2="43.18" y2="37.1983" width="0.6096" layer="1"/>
 <wire x1="37.7825" y1="60.325" x2="39.0525" y2="60.325" width="0.6096" layer="16"/>
 <wire x1="41.6433" y1="60.325" x2="43.18" y2="58.7883" width="0.6096" layer="16"/>
@@
 <wire x1="39.0525" y1="114.3" x2="46.6725" y2="114.3" width="1.27" layer="16"/>
 <wire x1="95.885" y1="114.3" x2="46.6725" y2="114.3" width="1.27" layer="16"/>
+<contactref element="JP3" pad="1"/>
+<wire x1="60.325" y1="27.6225" x2="60.325" y2="30.0736" width="0.6096" layer="16"/>
+<wire x1="60.325" y1="30.0736" x2="60.325" y2="38.4175" width="0.6096" layer="16"/>
+<wire x1="60.325" y1="38.4175" x2="59.69" y2="39.0525" width="0.6096" layer="16"/>
+<wire x1="59.69" y1="39.0525" x2="47.9425" y2="39.0525" width="0.6096" layer="16"/>
+<wire x1="47.9425" y1="39.0525" x2="47.625" y2="38.735" width="0.6096" layer="16"/>
+<wire x1="47.625" y1="38.735" x2="47.625" y2="37.1983" width="0.6096" layer="16"/>
+<contactref element="C7" pad="1"/>
+<wire x1="43.18" y1="24.7659" x2="44.7675" y2="24.7659" width="0.6096" layer="16"/>
+<wire x1="44.45" y1="21.32" x2="44.45" y2="24.423" width="0.4064" layer="16"/>
+<wire x1="44.45" y1="24.423" x2="44.7675" y2="24.7659" width="0.4064" layer="16"/>
+<wire x1="45.085" y1="21.32" x2="45.085" y2="24.4738" width="0.4064" layer="16"/>
+<wire x1="45.085" y1="24.4738" x2="44.7675" y2="24.7659" width="0.4064" layer="16"/>
 </signal>
 <signal name="GND">
@@
 <via x="135.5725" y="29.21" extent="1-16" drill="0.6" diameter="1.4224" shape="octagon"/>
 <wire x1="135.5725" y1="48.895" x2="135.5725" y2="29.21" width="0.6096" layer="1"/>
-<wire x1="41.275" y1="24.765" x2="41.275" y2="21.32" width="0.4064" layer="16"/>
-<wire x1="41.275" y1="24.765" x2="41.91" y2="25.4" width="0.4064" layer="16"/>
+<wire x1="41.275" y1="26.035" x2="41.275" y2="21.32" width="0.4064" layer="16"/>
+<wire x1="41.275" y1="26.035" x2="41.91" y2="26.67" width="0.4064" layer="16"/>
 <via x="61.2775" y="40.005" extent="1-16" drill="0.6" diameter="1.4224" shape="octagon"/>
 <via x="61.2775" y="46.99" extent="1-16" drill="0.6" diameter="1.4224" shape="octagon"/>
 <wire x1="61.2775" y1="40.005" x2="61.2775" y2="46.99" width="0.6096" layer="1"/>
+<contactref element="JP3" pad="2"/>
+<contactref element="C7" pad="2"/>
+<contactref element="C8" pad="1"/>
 </signal>
 <signal name="D0">
@@
 <via x="48.26" y="24.765" extent="1-16" drill="0.6" diameter="1.4224" shape="octagon"/>
 <contactref element="CON1" pad="35"/>
-<wire x1="48.26" y1="21.32" x2="48.26" y2="24.765" width="0.4064" layer="16"/>
 <wire x1="85.09" y1="22.225" x2="80.01" y2="22.225" width="0.4064" layer="16"/>
 <wire x1="80.01" y1="22.225" x2="78.74" y2="23.495" width="0.4064" layer="16"/>
@@
 <wire x1="62.5475" y1="24.765" x2="67.6275" y2="24.765" width="0.4064" layer="16"/>
 <wire x1="67.6275" y1="24.765" x2="68.8975" y2="23.495" width="0.4064" layer="16"/>
+<wire x1="48.26" y1="21.32" x2="48.26" y2="24.765" width="0.4064" layer="16"/>
 </signal>
 <signal name="MEM_WR">
@@
 <wire x1="31.75" y1="38.735" x2="35.052" y2="38.735" width="0.4064" layer="16"/>
 <wire x1="35.052" y1="38.735" x2="36.195" y2="39.878" width="0.4064" layer="16"/>
+<contactref element="C8" pad="2"/>
+<wire x1="36.195" y1="39.878" x2="37.885" y2="39.878" width="0.6096" layer="16"/>
 </signal>
 <signal name="N$8">
@@
 <via x="49.53" y="26.035" extent="1-16" drill="0.6" diameter="1.4224" shape="octagon"/>
 <contactref element="CON1" pad="34"/>
-<wire x1="49.53" y1="26.035" x2="49.53" y2="21.32" width="0.4064" layer="16"/>
 <wire x1="63.8175" y1="26.035" x2="78.74" y2="26.035" width="0.4064" layer="16"/>
 <wire x1="78.74" y1="26.035" x2="80.01" y2="24.765" width="0.4064" layer="16"/>
+<wire x1="49.53" y1="26.035" x2="49.53" y2="21.32" width="0.4064" layer="16"/>
 </signal>
 <signal name="A14_CPU">
@@
 <contactref element="CON1" pad="36"/>
 <contactref element="R7" pad="1"/>
-<wire x1="46.99" y1="21.32" x2="46.99" y2="24.5364" width="0.4064" layer="16"/>
-<wire x1="46.6843" y1="24.5364" x2="46.99" y2="24.5364" width="0.4064" layer="16"/>
+<wire x1="46.99" y1="21.32" x2="46.99" y2="25.4" width="0.4064" layer="16"/>
+<wire x1="46.99" y1="25.4" x2="51.6636" y2="30.0736" width="0.4064" layer="16"/>
+<wire x1="52.705" y1="30.0736" x2="51.6636" y2="30.0736" width="0.4064" layer="16"/>
 </signal>
 <signal name="N$13">
@@
 <contactref element="CON1" pad="32"/>
 <contactref element="R11" pad="1"/>
-<wire x1="47.9425" y1="27.305" x2="50.8" y2="27.305" width="0.4064" layer="16"/>
-<wire x1="50.8" y1="27.305" x2="52.07" y2="26.035" width="0.4064" layer="16"/>
-<wire x1="52.07" y1="26.035" x2="52.07" y2="21.32" width="0.4064" layer="16"/>
-<wire x1="47.9425" y1="27.305" x2="46.6843" y2="26.0468" width="0.4064" layer="16"/>
-<wire x1="46.6843" y1="26.035" x2="46.6843" y2="26.0468" width="0.4064" layer="16"/>
+<wire x1="52.07" y1="24.13" x2="52.07" y2="21.32" width="0.4064" layer="16"/>
+<wire x1="52.705" y1="27.6225" x2="52.705" y2="24.765" width="0.4064" layer="16"/>
+<wire x1="52.705" y1="24.765" x2="52.07" y2="24.13" width="0.4064" layer="16"/>
 </signal>
 <signal name="CF_D3">

Commit message: Minor update
Routing:
- net A7: track 198.3 -> 197.5 mm
Changed lines of the file:
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@@
 <contactref element="IC2" pad="12"/>
 <via x="61.9125" y="80.645" extent="1-16" drill="0.6" diameter="1.4224" shape="octagon"/>
-<wire x1="61.9125" y1="80.645" x2="61.9125" y2="57.785" width="0.4064" layer="1"/>
-<via x="61.9125" y="57.785" extent="1-16" drill="0.6" diameter="1.4224" shape="octagon"/>
-<wire x1="79.375" y1="57.785" x2="61.9125" y2="57.785" width="0.4064" layer="16"/>
+<wire x1="61.9125" y1="80.645" x2="61.9125" y2="59.055" width="0.4064" layer="1"/>
+<via x="61.9125" y="59.055" extent="1-16" drill="0.6" diameter="1.4224" shape="octagon"/>
 <wire x1="35.56" y1="81.915" x2="36.83" y2="81.915" width="0.4064" layer="16"/>
 <wire x1="36.83" y1="81.915" x2="38.1" y2="80.645" width="0.4064" layer="16"/>
 <wire x1="38.1" y1="80.645" x2="61.9125" y2="80.645" width="0.4064" layer="16"/>
+<wire x1="61.9125" y1="59.055" x2="75.565" y2="59.055" width="0.4064" layer="16"/>
+<wire x1="75.565" y1="59.055" x2="76.835" y2="57.785" width="0.4064" layer="16"/>
+<wire x1="76.835" y1="57.785" x2="79.375" y2="57.785" width="0.4064" layer="16"/>
 </signal>
 <signal name="A8">
