File: hardware/8085.sch (EAGLE design)
At the start: 34 parts, among them IC2 74AC573N, IC3 ATF16V8BP3, IC4 74HCT245N, IC5 74HCT245DW, IC9 74HCT138N

Commit message: PCB updated
Parts:
- removed IC4: 74HCT245N, 74xx-eu:74HCT245N
- added Q1: (no value), crystal:CRYSTALHC49S
Connections:
- new net N$1: IC1.X1, Q1.2
- new net N$2: IC1.X2, Q1.1
- net D0: no longer IC4A.A1
- net D1: no longer IC4A.A2
- net D2: no longer IC4A.A3
- net D3: no longer IC4A.A4
- net D4: no longer IC4A.A5
- net D5: no longer IC4A.A6
- net D6: no longer IC4A.A7
- net D7: no longer IC4A.A8
Changed lines of the file:
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@@
 <part name="GND2" library="supply1" deviceset="GND" device=""/>
 <part name="IC1" library="micro-intel" deviceset="8085" device=""/>
-<part name="IC4" library="74xx-eu" deviceset="74*245" device="N" technology="HCT"/>
 <part name="IC2" library="74xx-eu" deviceset="74*573" device="N" technology="AC"/>
 <part name="GND1" library="supply1" deviceset="GND" device=""/>
@@
 <part name="IC5" library="74xx-eu" deviceset="74*245" device="DW" technology="HCT" value="74HCT245DW"/>
 <part name="GND8" library="supply1" deviceset="GND" device=""/>
+<part name="Q1" library="crystal" deviceset="CRYSTAL" device="HC49S"/>
 </parts>
 <sheets>
@@
 <instance part="GND2" gate="1" x="45.72" y="-111.76"/>
 <instance part="IC1" gate="G$1" x="10.16" y="22.86"/>
-<instance part="IC4" gate="A" x="10.16" y="175.26"/>
 <instance part="IC2" gate="A" x="10.16" y="129.54"/>
 <instance part="GND1" gate="1" x="-5.08" y="111.76"/>
@@
 <instance part="IC5" gate="A" x="10.16" y="223.52" rot="MR0"/>
 <instance part="GND8" gate="1" x="25.4" y="203.2"/>
+<instance part="Q1" gate="G$1" x="-17.78" y="7.62" rot="R90"/>
 </instances>
 <busses>
@@
 </segment>
 <segment>
-<pinref part="IC4" gate="A" pin="A1"/>
-<wire x1="-2.54" y1="187.96" x2="-7.62" y2="187.96" width="0.1524" layer="91"/>
-<label x="-7.62" y="187.96" size="1.4224" layer="95" rot="R180" xref="yes"/>
-</segment>
-<segment>
 <pinref part="IC2" gate="A" pin="1D"/>
 <wire x1="-2.54" y1="142.24" x2="-7.62" y2="142.24" width="0.1524" layer="91"/>
@@
 </segment>
 <segment>
-<pinref part="IC4" gate="A" pin="A2"/>
-<wire x1="-2.54" y1="185.42" x2="-7.62" y2="185.42" width="0.1524" layer="91"/>
-<label x="-7.62" y="185.42" size="1.4224" layer="95" rot="R180" xref="yes"/>
-</segment>
-<segment>
 <pinref part="IC2" gate="A" pin="2D"/>
 <wire x1="-2.54" y1="139.7" x2="-7.62" y2="139.7" width="0.1524" layer="91"/>
@@
 </segment>
 <segment>
-<pinref part="IC4" gate="A" pin="A3"/>
-<wire x1="-2.54" y1="182.88" x2="-7.62" y2="182.88" width="0.1524" layer="91"/>
-<label x="-7.62" y="182.88" size="1.4224" layer="95" rot="R180" xref="yes"/>
-</segment>
-<segment>
 <pinref part="IC2" gate="A" pin="3D"/>
 <wire x1="-2.54" y1="137.16" x2="-7.62" y2="137.16" width="0.1524" layer="91"/>
@@
 </segment>
 <segment>
-<pinref part="IC4" gate="A" pin="A4"/>
-<wire x1="-2.54" y1="180.34" x2="-7.62" y2="180.34" width="0.1524" layer="91"/>
-<label x="-7.62" y="180.34" size="1.4224" layer="95" rot="R180" xref="yes"/>
-</segment>
-<segment>
 <pinref part="IC2" gate="A" pin="4D"/>
 <wire x1="-2.54" y1="134.62" x2="-7.62" y2="134.62" width="0.1524" layer="91"/>
@@
 </segment>
 <segment>
-<pinref part="IC4" gate="A" pin="A5"/>
-<wire x1="-2.54" y1="177.8" x2="-7.62" y2="177.8" width="0.1524" layer="91"/>
-<label x="-7.62" y="177.8" size="1.4224" layer="95" rot="R180" xref="yes"/>
-</segment>
-<segment>
 <pinref part="IC2" gate="A" pin="5D"/>
 <wire x1="-2.54" y1="132.08" x2="-7.62" y2="132.08" width="0.1524" layer="91"/>
@@
 </segment>
 <segment>
-<pinref part="IC4" gate="A" pin="A6"/>
-<wire x1="-2.54" y1="175.26" x2="-7.62" y2="175.26" width="0.1524" layer="91"/>
-<label x="-7.62" y="175.26" size="1.4224" layer="95" rot="R180" xref="yes"/>
-</segment>
-<segment>
 <pinref part="IC2" gate="A" pin="6D"/>
 <wire x1="-2.54" y1="129.54" x2="-7.62" y2="129.54" width="0.1524" layer="91"/>
@@
 </segment>
 <segment>
-<pinref part="IC4" gate="A" pin="A7"/>
-<wire x1="-2.54" y1="172.72" x2="-5.08" y2="172.72" width="0.1524" layer="91"/>
-<wire x1="-7.62" y1="172.72" x2="-5.08" y2="172.72" width="0.1524" layer="91"/>
-<label x="-7.62" y="172.72" size="1.4224" layer="95" rot="R180" xref="yes"/>
-</segment>
-<segment>
 <pinref part="IC2" gate="A" pin="7D"/>
 <wire x1="-2.54" y1="127" x2="-7.62" y2="127" width="0.1524" layer="91"/>
@@
 <wire x1="25.4" y1="43.18" x2="30.48" y2="43.18" width="0.1524" layer="91"/>
 <label x="30.48" y="43.18" size="1.4224" layer="95" xref="yes"/>
-</segment>
-<segment>
-<pinref part="IC4" gate="A" pin="A8"/>
-<wire x1="-2.54" y1="170.18" x2="-7.62" y2="170.18" width="0.1524" layer="91"/>
-<label x="-7.62" y="170.18" size="1.4224" layer="95" rot="R180" xref="yes"/>
 </segment>
 <segment>
@@
 </segment>
 </net>
+<net name="N$1" class="0">
+<segment>
+<pinref part="IC1" gate="G$1" pin="X1"/>
+<wire x1="-7.62" y1="10.16" x2="-12.7" y2="10.16" width="0.1524" layer="91"/>
+<wire x1="-12.7" y1="10.16" x2="-12.7" y2="12.7" width="0.1524" layer="91"/>
+<pinref part="Q1" gate="G$1" pin="2"/>
+<wire x1="-12.7" y1="12.7" x2="-17.78" y2="12.7" width="0.1524" layer="91"/>
+<wire x1="-17.78" y1="12.7" x2="-17.78" y2="10.16" width="0.1524" layer="91"/>
+</segment>
+</net>
+<net name="N$2" class="0">
+<segment>
+<pinref part="IC1" gate="G$1" pin="X2"/>
+<wire x1="-7.62" y1="5.08" x2="-12.7" y2="5.08" width="0.1524" layer="91"/>
+<wire x1="-12.7" y1="5.08" x2="-12.7" y2="2.54" width="0.1524" layer="91"/>
+<pinref part="Q1" gate="G$1" pin="1"/>
+<wire x1="-12.7" y1="2.54" x2="-17.78" y2="2.54" width="0.1524" layer="91"/>
+<wire x1="-17.78" y1="2.54" x2="-17.78" y2="5.08" width="0.1524" layer="91"/>
+</segment>
+</net>

Commit message: PCB updated
Parts:
- removed LED1, LED2: (no value), led:LED3MM
- removed R1: 1k, rcl:R-EU_M1206
- removed R7, R8: 470R, rcl:R-EU_R0603
- removed U$1: UCY74S412, mw:UCY74S412
- added IC10: 74HCT00N, 74xx-eu:74HCT00N
- added IC4: 74AC00D, 74xx-eu:74AC00D
- added IC6: 74AC273N, 74xx-eu:74AC273N
- added IC7: 74HCT139N, 74xx-eu:74HCT139N
- added IC8: 7404N, 74xx-us:7404N
- added LED3, LED4: (no value), led:LED5MM
- added R2, R3: (no value), rcl:R-EU_R1206
- C1, C14, C2, C3, C6: device rcl:C-EUC1206 -> rcl:C-EUC0805
- R9: device rcl:R-EU_0204/7 -> rcl:R-EU_M1206
Connections:
- net HALT renamed HRQ
- removed net !CS_PORT_OUT: U$1.DS2
- removed net !IORQ: IC3.I3, IC9A.G2A
- removed net !MREQ: IC3.CLK
- removed net A14_IN: IC1.A14, IC5A.B2
- removed net A15_IN: IC1.A15, IC5A.B1
- removed net BUSAK: SV2.38
- removed net BUSRQ: SV2.37
- removed net CS_RAM1: IC3.O1, U$4.!CS
- removed net DMA_CS: IC3.O6
- removed net DMA_RDY: SV2.40
- removed net M1: IC3.I4
- removed net N$17: LED2.C, R8.2
- removed net N$3: R7.1, U$1.DO6
- removed net N$4: LED1.C, R7.2
- removed net N$6: R8.1, U$1.DO7
- removed net N$7: R1.2, U$1.!MD
- removed net NMI: SV2.39
- removed net PORT_CS: IC3.O5
- removed net ROM_SHADOWING: IC3.I1, U$1.DO2
- removed net WAIT: SV2.42
- new net !A15: IC7A.G, IC8A.O
- new net A14_CPU: IC1.A14, IC4C.I0, IC4C.I1
- new net A14_SWITCH: IC4B.O, IC5A.B2
- new net A15_CPU: IC1.A15, IC4D.I0, IC4D.I1
- new net A15_SWITCH: IC4A.O, IC5A.B1
- new net AEN: IC2A.OC, IC5A.G, IC9A.G2A, SV2.42
- new net BANK_A14: IC10B.O, U$2.A14
- new net IO_M: IC1.IO/!M, IC3.I3
- new net IO_RD: IC3.O1, SV2.34
- new net IO_WR: IC3.O2, SV2.35
- new net MEM_RD: IC3.O3, SV2.39, U$2.!OE, U$3.!RD, U$4.!OE
- new net MEM_WR: IC3.O4, SV2.40, U$2.!WE, U$4.!WE
- new net N$10: IC6A.Q8, R2.1
- new net N$19: IC7A.Y0, IC7B.G
- new net N$21: IC4B.I1, IC4C.O
- new net N$26: IC4A.I0, IC4D.O
- new net N$5: IC6A.Q7, R3.1
- new net N$8: LED3.C, R2.2
- new net N$9: LED4.C, R3.2
- new net RESET: IC1.RES_OUT, IC8B.I, SV2.37
- new net START_MEM_SWITCH: IC4A.I1, IC4B.I0, IC6A.Q3
- net !RESET: now also IC6A.CLR, IC8B.O; no longer U$1.!CLR
- net 8275_DACK: now also IC10B.I1
- net A13: now also IC7B.A
- net A14: now also IC7A.A; no longer U$2.A14
- net A15: now also IC8A.I, U$4.!CS; no longer IC3.I2
- net A4: no longer IC3.I6
- net CS_EPROM: now also IC7A.Y1; no longer IC3.O3
- net CS_RAM2: now also IC7B.Y0; no longer IC3.O2
- net D0: now also IC6A.D1; no longer U$1.DI0
- net D1: now also IC6A.D2; no longer U$1.DI1
- net D2: now also IC6A.D3; no longer U$1.DI2
- net D3: now also IC6A.D4; no longer U$1.DI3
- net D4: now also IC6A.D5; no longer U$1.DI4
- net D5: now also IC6A.D6; no longer U$1.DI5
- net D6: now also IC6A.D7; no longer U$1.DI6
- net D7: now also IC6A.D8; no longer U$1.DI7
- net GND: now also IC10A.I0, IC10A.I1, IC10C.I0, IC10C.I1, IC10D.I0, IC10D.I1, IC10P.GND, IC7A.B, IC7B.B, IC8C.I, IC8D.I, IC8E.I, IC8F.I, IC8P.GND; no longer IC2A.OC, IC3.GND, IC5A.G, U$1.GND
- net HLDA: now also SV2.38
- net INT: now also IC1.INTR
- net INTA: now also IC1.INTA; no longer IC3.O4
- net LOCAL_IO_CS: no longer IC3.I5
- net OUT_1: now also IC6A.Q5; no longer U$1.DO4
- net OUT_2: now also IC6A.Q6; no longer U$1.DO5
- net OUT_3: now also IC6A.Q4; no longer U$1.DO3
- net OUT_4: now also IC6A.Q2; no longer U$1.DO1
- net RD: now also IC3.I2; no longer SV2.34, U$2.!OE, U$3.!RD, U$4.!OE
- net SET_BANK_A14: now also IC10B.I0, IC6A.Q1; no longer U$1.DO0
- net VCC: now also IC10P.VCC, IC8P.VCC, LED3.A, LED4.A; no longer IC3.VCC, LED1.A, LED2.A, R1.1, U$1.VCC
- net WR: now also IC3.I1; no longer SV2.35, U$1.DS1, U$2.!WE, U$4.!WE

Commit message: PCB updated
Parts:
- added IC11: 74HCT245DW, 74xx-eu:74HCT245DW
- added IC12: DS1813, ds1813_revised:DS1813
- added JP1: (no value), pinhead:PINHD-1X2
- added R1, R4, R5, R6: (no value), rcl:R-EU_R0603
- added SV1: (no value), con-ml:ML40
- C21: device rcl:C-EUC1206 -> rcl:C-EUC0603
Connections:
- removed net HOLD: IC1.HOLD
- new net CF_BDV2_LED: SV1.39
- new net CF_BVD1: SV1.34
- new net CF_CE1: SV1.37
- new net CF_CE2: SV1.38
- new net CF_INPACK: SV1.21
- new net CF_RDY_CSY_IREQ: SV1.31
- new net CF_REG: SV1.29
- new net CF_WAIT: SV1.27
- new net CF_WP_IOCS16: SV1.32
- new net D0_CF: IC11A.B1, SV1.17
- new net D1_CF: IC11A.B2, SV1.15
- new net D2_CF: IC11A.B3, SV1.13
- new net D3_CF: IC11A.B4, SV1.11
- new net D4_CF: IC11A.B5, SV1.9
- new net D5_CF: IC11A.B6, SV1.7
- new net D6_CF: IC11A.B7, SV1.5
- new net D7_CF: IC11A.B8, SV1.3
- new net LOCAL_PORT_CS: IC3.O5, IC6A.CLK
- new net N$3: IC1.RST5_5, R1.1
- new net N$4: IC1.RST6_5, R4.1
- new net N$6: IC1.RST7_5, R5.1
- new net N$7: IC1.TRAP, R6.1
- new net RES_IN: IC1.RES_IN, IC12./RST, JP1.2
- net !RESET: now also SV1.1
- net A0: now also SV1.35
- net A1: now also SV1.33
- net A2: now also SV1.36
- net A4: now also IC3.I1
- net D0: now also IC11A.A1
- net D1: now also IC11A.A2
- net D2: now also IC11A.A3
- net D3: now also IC11A.A4
- net D4: now also IC11A.A5
- net D5: now also IC11A.A6
- net D6: now also IC11A.A7
- net D7: now also IC11A.A8
- net GND: now also IC12.GND, JP1.1, R1.2, R4.2, R5.2, R6.2, SV1.19, SV1.2, SV1.22, SV1.24, SV1.26
- net HRQ: now also IC1.HOLD
- net IO_M: now also IC3.I2; no longer IC3.I3
- net IO_RD: now also SV1.25
- net IO_WR: now also SV1.23
- net LOCAL_IO_CS: now also IC3.I5
- net RD: now also IC3.I3; no longer IC3.I2
- net RDYIN: now also IC1.READY
- net VCC: now also IC12.+5V
- net WR: now also IC3.I4; no longer IC3.I1

Commit message: Reset circuit simplified
Parts:
- removed IC12: DS1813, ds1813_revised:DS1813
- removed R5, R6: (no value), rcl:R-EU_R0603
- removed SV1: (no value), con-ml:ML40
- added C4: (no value), rcl:C-EUC0603
- added CON1: (no value), con-hirose:CF-CARD-IDE_MODE
- added D1: 1N4148DO35-7, diode:1N4148DO35-7
- added R10, R11, R7: (no value), rcl:R-EU_R0603
- added R8: (no value), rcl:R-EU_0204/7
- added RN1: (no value), resistor-sil:G04R
- R1, R4: device rcl:R-EU_R0603 -> rcl:R-EU_0204/7
Connections:
- removed net CF_BDV2_LED: SV1.39
- removed net CF_BVD1: SV1.34
- removed net CF_CE1: SV1.37
- removed net CF_CE2: SV1.38
- removed net CF_INPACK: SV1.21
- removed net CF_RDY_CSY_IREQ: SV1.31
- removed net CF_REG: SV1.29
- removed net CF_WAIT: SV1.27
- removed net CF_WP_IOCS16: SV1.32
- removed net D0_CF: IC11A.B1, SV1.17
- removed net D1_CF: IC11A.B2, SV1.15
- removed net D2_CF: IC11A.B3, SV1.13
- removed net D3_CF: IC11A.B4, SV1.11
- removed net D4_CF: IC11A.B5, SV1.9
- removed net D5_CF: IC11A.B6, SV1.7
- removed net D6_CF: IC11A.B7, SV1.5
- removed net D7_CF: IC11A.B8, SV1.3
- new net CF_CS0: CON1G$1./CS0
- new net CF_D0: CON1G$1.D00, IC11A.B1
- new net CF_D1: CON1G$1.D01, IC11A.B2
- new net CF_D2: CON1G$1.D02, IC11A.B3
- new net CF_D3: CON1G$1.D03, IC11A.B8
- new net CF_D4: CON1G$1.D04, IC11A.B7
- new net CF_D5: CON1G$1.D05, IC11A.B6
- new net CF_D6: CON1G$1.D06, IC11A.B5
- new net CF_D7: CON1G$1.D07, IC11A.B4
- new net N$11: CON1G$1./REG, R8.1
- new net N$12: CON1G$1./WE, R7.1
- new net N$13: CON1G$1./PDIAG, R10.1
- new net N$14: JP1.2, R1.1
- new net N$29: CON1G$1./CS1, R11.1
- net !RESET: now also CON1G$1./RESET; no longer SV1.1
- net A0: now also CON1G$1.A00; no longer SV1.35
- net A1: now also CON1G$1.A01; no longer SV1.33
- net A2: now also CON1G$1.A02; no longer SV1.36
- net D3: now also IC11A.A8; no longer IC11A.A4
- net D4: now also IC11A.A7; no longer IC11A.A5
- net D6: now also IC11A.A5; no longer IC11A.A7
- net D7: now also IC11A.A4; no longer IC11A.A8
- net GND: now also C4.2, CON1G$1./ATASEL, CON1G$1./CSEL, CON1G$1.A03, CON1G$1.A04, CON1G$1.A05, CON1G$1.A06, CON1G$1.A07, CON1G$1.A08, CON1G$1.A09, CON1G$1.A10, CON1P.GND1, CON1P.GND2; no longer IC12.GND, R1.2, R4.2, R5.2, R6.2, SV1.19, SV1.2, SV1.22, SV1.24, SV1.26
- net IO_RD: now also CON1G$1./IORD; no longer SV1.25
- net IO_WR: now also CON1G$1./IOWR; no longer SV1.23
- net N$3: now also RN1.2; no longer R1.1
- net N$4: now also RN1.3; no longer R4.1
- net N$6: now also RN1.4; no longer R5.1
- net N$7: now also RN1.5; no longer R6.1
- net RES_IN: now also C4.1, D1.A, R1.2, R4.1; no longer IC12./RST, JP1.2
- net VCC: now also CON1P.VCC1, CON1P.VCC2, D1.C, R10.2, R11.2, R4.2, R7.2, R8.2, RN1.1; no longer IC12.+5V
Other:
- moved on the sheet: JP1, R1, R4

Commit message: Minor optimizations
Connections:
- net GND: now also RN1.1
- net VCC: no longer RN1.1
Changed lines of the file:
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@@
 <part name="R4" library="rcl" deviceset="R-EU_" device="0204/7"/>
 <part name="C4" library="rcl" deviceset="C-EU" device="C0603"/>
+<part name="GND16" library="supply1" deviceset="GND" device=""/>
 </parts>
 <sheets>
@@
 <instance part="R4" gate="G$1" x="-86.36" y="71.12" rot="R90"/>
 <instance part="C4" gate="G$1" x="-86.36" y="53.34"/>
+<instance part="GND16" gate="1" x="-43.18" y="43.18"/>
 </instances>
 <busses>
@@
 <label x="248.92" y="-259.08" size="1.4224" layer="95" rot="R90" xref="yes"/>
 </segment>
-<segment>
-<pinref part="RN1" gate="A" pin="1"/>
-<wire x1="-35.56" y1="50.8" x2="-35.56" y2="55.88" width="0.1524" layer="91"/>
-</segment>
 </net>
 <net name="GND" class="0">
@@
 <wire x1="-86.36" y1="40.64" x2="-86.36" y2="48.26" width="0.1524" layer="91"/>
 </segment>
+<segment>
+<pinref part="RN1" gate="A" pin="1"/>
+<wire x1="-35.56" y1="50.8" x2="-35.56" y2="53.34" width="0.1524" layer="91"/>
+<wire x1="-35.56" y1="53.34" x2="-43.18" y2="53.34" width="0.1524" layer="91"/>
+<wire x1="-43.18" y1="53.34" x2="-43.18" y2="45.72" width="0.1524" layer="91"/>
+<pinref part="GND16" gate="1" pin="GND"/>
+</segment>
 </net>

Commit message: PCB design upadted
Parts:
- C5: device rcl:C-EU050-024X044 -> rcl:C-EUC0603
- R1: device rcl:R-EU_0204/7 -> rcl:R-EU_0204/5
- R10: device rcl:R-EU_R0603 -> rcl:R-EU_0207/10
- R8: device rcl:R-EU_0204/7 -> rcl:R-EU_0207/10
Connections:
- net CF_D0: now also IC11A.B3; no longer IC11A.B1
- net CF_D2: now also IC11A.B1; no longer IC11A.B3
- net D0: now also IC11A.A3; no longer IC11A.A1
- net D2: now also IC11A.A1; no longer IC11A.A3
- net IO_M: now also IC3.I5; no longer IC3.I2
- net LOCAL_IO_CS: now also IC3.I6; no longer IC3.I5
Changed lines of the file:
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@@
 <part name="C3" library="rcl" deviceset="C-EU" device="C0805" value="100n"/>
 <part name="GND6" library="supply1" deviceset="GND" device=""/>
-<part name="C5" library="rcl" deviceset="C-EU" device="050-024X044" value="100n"/>
+<part name="C5" library="rcl" deviceset="C-EU" device="C0603" value="100n"/>
 <part name="C6" library="rcl" deviceset="C-EU" device="C0805" value="100n"/>
 <part name="IC9" library="74xx-eu" deviceset="74*138" device="N" technology="HCT"/>
@@
 <part name="GND20" library="supply1" deviceset="GND" device=""/>
 <part name="R7" library="rcl" deviceset="R-EU_" device="R0603"/>
-<part name="R8" library="rcl" deviceset="R-EU_" device="0204/7"/>
-<part name="R10" library="rcl" deviceset="R-EU_" device="R0603"/>
+<part name="R8" library="rcl" deviceset="R-EU_" device="0207/10"/>
+<part name="R10" library="rcl" deviceset="R-EU_" device="0207/10"/>
 <part name="R11" library="rcl" deviceset="R-EU_" device="R0603"/>
 <part name="RN1" library="resistor-sil" deviceset="G04R" device=""/>
-<part name="R1" library="rcl" deviceset="R-EU_" device="0204/7"/>
+<part name="R1" library="rcl" deviceset="R-EU_" device="0204/5"/>
 <part name="D1" library="diode" deviceset="1N4148" device="DO35-7"/>
 <part name="R4" library="rcl" deviceset="R-EU_" device="0204/7"/>
@@
 </segment>
 <segment>
-<pinref part="IC11" gate="A" pin="A1"/>
-<wire x1="106.68" y1="-297.18" x2="114.3" y2="-297.18" width="0.1524" layer="91"/>
-<label x="114.3" y="-297.18" size="1.4224" layer="95" xref="yes"/>
+<pinref part="IC11" gate="A" pin="A3"/>
+<wire x1="106.68" y1="-302.26" x2="111.76" y2="-302.26" width="0.1524" layer="91"/>
+<label x="111.76" y="-302.26" size="1.4224" layer="95" xref="yes"/>
 </segment>
 </net>
@@
 <segment>
 <pinref part="IC11" gate="A" pin="A2"/>
-<wire x1="106.68" y1="-299.72" x2="114.3" y2="-299.72" width="0.1524" layer="91"/>
-<label x="114.3" y="-299.72" size="1.4224" layer="95" xref="yes"/>
+<wire x1="106.68" y1="-299.72" x2="111.76" y2="-299.72" width="0.1524" layer="91"/>
+<label x="111.76" y="-299.72" size="1.4224" layer="95" xref="yes"/>
 </segment>
 </net>
@@
 </segment>
 <segment>
-<pinref part="IC11" gate="A" pin="A3"/>
-<wire x1="106.68" y1="-302.26" x2="114.3" y2="-302.26" width="0.1524" layer="91"/>
-<label x="114.3" y="-302.26" size="1.4224" layer="95" xref="yes"/>
+<pinref part="IC11" gate="A" pin="A1"/>
+<wire x1="106.68" y1="-297.18" x2="111.76" y2="-297.18" width="0.1524" layer="91"/>
+<label x="111.76" y="-297.18" size="1.4224" layer="95" xref="yes"/>
 </segment>
 </net>
@@
 </segment>
 <segment>
-<pinref part="IC3" gate="G$1" pin="I5"/>
-<wire x1="48.26" y1="-93.98" x2="43.18" y2="-93.98" width="0.1524" layer="91"/>
-<label x="43.18" y="-93.98" size="1.4224" layer="95" rot="R180" xref="yes"/>
+<pinref part="IC3" gate="G$1" pin="I6"/>
+<wire x1="48.26" y1="-96.52" x2="43.18" y2="-96.52" width="0.1524" layer="91"/>
+<label x="43.18" y="-96.52" size="1.4224" layer="95" rot="R180" xref="yes"/>
 </segment>
 </net>
@@
 </segment>
 <segment>
-<pinref part="IC3" gate="G$1" pin="I2"/>
-<wire x1="48.26" y1="-86.36" x2="43.18" y2="-86.36" width="0.1524" layer="91"/>
-<label x="43.18" y="-86.36" size="1.4224" layer="95" rot="R180" xref="yes"/>
+<pinref part="IC3" gate="G$1" pin="I5"/>
+<wire x1="48.26" y1="-93.98" x2="43.18" y2="-93.98" width="0.1524" layer="91"/>
+<label x="43.18" y="-93.98" size="1.4224" layer="95" rot="R180" xref="yes"/>
 </segment>
 </net>
@@
 <net name="CF_D2" class="0">
 <segment>
-<pinref part="IC11" gate="A" pin="B3"/>
-<wire x1="81.28" y1="-302.26" x2="76.2" y2="-302.26" width="0.1524" layer="91"/>
-</segment>
-<segment>
 <pinref part="CON1" gate="G$1" pin="D02"/>
 <wire x1="241.3" y1="-233.68" x2="246.38" y2="-233.68" width="0.1524" layer="91"/>
 <label x="246.38" y="-233.68" size="1.4224" layer="95" xref="yes"/>
 </segment>
+<segment>
+<pinref part="IC11" gate="A" pin="B1"/>
+<wire x1="81.28" y1="-297.18" x2="76.2" y2="-297.18" width="0.1524" layer="91"/>
+<label x="76.2" y="-297.18" size="1.4224" layer="95" rot="R180" xref="yes"/>
+</segment>
 </net>
 <net name="CF_D1" class="0">
@@
 <pinref part="IC11" gate="A" pin="B2"/>
 <wire x1="81.28" y1="-299.72" x2="76.2" y2="-299.72" width="0.1524" layer="91"/>
+<label x="76.2" y="-299.72" size="1.4224" layer="95" rot="R180" xref="yes"/>
 </segment>
 <segment>
@@
 <net name="CF_D0" class="0">
 <segment>
-<pinref part="IC11" gate="A" pin="B1"/>
-<wire x1="81.28" y1="-297.18" x2="76.2" y2="-297.18" width="0.1524" layer="91"/>
-</segment>
-<segment>
 <pinref part="CON1" gate="G$1" pin="D00"/>
 <wire x1="241.3" y1="-228.6" x2="246.38" y2="-228.6" width="0.1524" layer="91"/>
 <label x="246.38" y="-228.6" size="1.4224" layer="95" xref="yes"/>
 </segment>
-</net>
+<segment>
+<pinref part="IC11" gate="A" pin="B3"/>
+<wire x1="81.28" y1="-302.26" x2="76.2" y2="-302.26" width="0.1524" layer="91"/>
+<label x="76.2" y="-302.26" size="1.4224" layer="95" rot="R180" xref="yes"/>
+</segment>
+</net>

Commit message: Minor PCB updates
Parts:
- added C7: 100n, rcl:C-EUC0603
- added C8: 22p, rcl:C-EUC0603
- added JP3: (no value), pinhead:PINHD-1X2
- R11, R7: device rcl:R-EU_R0603 -> rcl:R-EU_0204/7
Connections:
- net GND: now also C7.2, C8.1, JP3.2
- net N$2: now also C8.2
- net VCC: now also C7.1, JP3.1
