File: hardware/8085.sch (EAGLE design)
At the start: 53 parts, among them IC10 74HCT00N, IC11 74HCT245DW, IC2 74AC573N, IC3 ATF16V8BP3, IC4 74AC00D, IC5 74HCT245DW, IC6 74AC273N, IC7 74HCT139N, IC8 7404N, IC9 74HCT138N

Commit message: Bugs in PCB board fixed
Parts:
- removed C12: 100n, rcl:C-EUC0805
- removed IC8: 7404N, 74xx-us:7404N
- added R12, R13, R9: (no value), rcl:R-EU_R0603
- added R14: (no value), rcl:R-EU_0204/7
- added R6: (no value), rcl:R-EU_0204/5
- IC2: value 74AC573N -> 74HCT574N; device 74xx-eu:74AC573N -> 74xx-eu:74HCT574N
Connections:
- removed net !A15: IC7A.G, IC8A.O
- removed net IO_RD: CON1G$1./IORD, IC11A.DIR, IC3.O1, SV2.34
- removed net IO_WR: CON1G$1./IOWR, IC3.O2, SV2.35
- removed net MEM_RD: IC3.O3, SV2.39, U$2.!OE, U$3.!RD, U$4.!OE
- removed net MEM_WR: IC3.O4, SV2.40, U$2.!WE, U$4.!WE
- new net !ALE: IC10A.O, IC2A.CLK
- new net CF_DELAYED_RD: CON1G$1./IORD, IC3.O1
- new net CF_DELAYED_WR: CON1G$1./IOWR, IC3.O2
- new net CS_RAM1: IC7A.Y0, U$4.!CS
- new net MEM_EN: IC3.O4, IC7A.G
- net !RESET: now also IC3.O6; no longer IC8B.O
- net 8275_DACK: now also R14.1
- net A13: no longer IC7B.A
- net A14: now also IC7B.A; no longer IC7A.A
- net A15: now also IC7A.A; no longer IC8A.I, U$4.!CS
- net AEN: now also IC3.I7, R9.1
- net ALE: now also IC10A.I0, IC10A.I1; no longer IC2A.C, IC3.I2
- net CF_CS0: now also IC3.O3; no longer IC3.O6
- net CS_EPROM: now also IC7B.Y1; no longer IC7A.Y1
- net GND: now also R12.1, R13.1, R9.2, SV2.40; no longer C12.2, IC10A.I0, IC10A.I1, IC3.I7, IC8C.I, IC8D.I, IC8E.I, IC8F.I, IC8P.GND
- net HRQ: now also R12.2
- net INT: now also R13.2
- net IO_M: now also SV2.39
- net N$19: now also IC7A.Y1; no longer IC7A.Y0
- net RD: now also IC11A.DIR, SV2.34, U$2.!OE, U$3.!RD, U$4.!OE
- net RDYIN: now also R6.1
- net RESET: now also IC3.I2; no longer IC8B.I
- net VCC: now also R14.2, R6.2; no longer C12.1, IC8P.VCC
- net WR: now also SV2.35, U$2.!WE, U$4.!WE
Other:
- moved on the sheet: C13, C14, C15, C18, C21, C22, C7, RN1

Commit message: CPU board updated
Parts:
- R5: device rcl:R-EU_M1206 -> rcl:R-EU_R0603
Changed lines of the file:
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@@
 <part name="GND17" library="supply1" deviceset="GND" device=""/>
 <part name="GND18" library="supply1" deviceset="GND" device=""/>
-<part name="R5" library="rcl" deviceset="R-EU_" device="M1206"/>
+<part name="R5" library="rcl" deviceset="R-EU_" device="R0603"/>
 <part name="LED1" library="led" deviceset="LED" device="5MM"/>
 <part name="R6" library="rcl" deviceset="R-EU_" device="0204/5"/>

Commit message: Small changes in PCB design
Parts:
- added R15, R16: (no value), rcl:R-EU_0204/7
- added R17: (no value), rcl:R-EU_0207/10
Connections:
- net !RESET: now also R17.2
- net RD: now also R15.1
- net VCC: now also R15.2, R16.2, R17.1
- net WR: now also R16.1
Changed lines of the file:
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@@
 <part name="R14" library="rcl" deviceset="R-EU_" device="0204/7"/>
 <part name="GND10" library="supply1" deviceset="GND" device=""/>
+<part name="R15" library="rcl" deviceset="R-EU_" device="0204/7"/>
+<part name="R16" library="rcl" deviceset="R-EU_" device="0204/7"/>
+<part name="R17" library="rcl" deviceset="R-EU_" device="0207/10"/>
 </parts>
 <sheets>
@@
 <instance part="R14" gate="G$1" x="327.66" y="-119.38" rot="R90"/>
 <instance part="GND10" gate="1" x="48.26" y="-157.48"/>
+<instance part="R15" gate="G$1" x="45.72" y="7.62" rot="R90"/>
+<instance part="R16" gate="G$1" x="50.8" y="7.62" rot="R90"/>
+<instance part="R17" gate="G$1" x="73.66" y="-109.22" rot="R90"/>
 </instances>
 <busses>
@@
 <label x="327.66" y="-111.76" size="1.4224" layer="95" rot="R90" xref="yes"/>
 </segment>
+<segment>
+<pinref part="R15" gate="G$1" pin="2"/>
+<wire x1="45.72" y1="12.7" x2="45.72" y2="15.24" width="0.1524" layer="91"/>
+<pinref part="R16" gate="G$1" pin="2"/>
+<wire x1="45.72" y1="15.24" x2="48.26" y2="15.24" width="0.1524" layer="91"/>
+<wire x1="48.26" y1="15.24" x2="50.8" y2="15.24" width="0.1524" layer="91"/>
+<wire x1="50.8" y1="15.24" x2="50.8" y2="12.7" width="0.1524" layer="91"/>
+<wire x1="48.26" y1="15.24" x2="48.26" y2="17.78" width="0.1524" layer="91"/>
+<junction x="48.26" y="15.24"/>
+<label x="48.26" y="17.78" size="1.4224" layer="95" rot="R90" xref="yes"/>
+</segment>
+<segment>
+<pinref part="R17" gate="G$1" pin="1"/>
+<wire x1="73.66" y1="-114.3" x2="73.66" y2="-116.84" width="0.1524" layer="91"/>
+<label x="73.66" y="-116.84" size="1.4224" layer="95" rot="R270" xref="yes"/>
+</segment>
 </net>
 <net name="GND" class="0">
@@
 <segment>
 <pinref part="IC3" gate="G$1" pin="O6"/>
-<wire x1="68.58" y1="-96.52" x2="76.2" y2="-96.52" width="0.1524" layer="91"/>
+<wire x1="68.58" y1="-96.52" x2="73.66" y2="-96.52" width="0.1524" layer="91"/>
 <label x="76.2" y="-96.52" size="1.4224" layer="95" xref="yes"/>
+<pinref part="R17" gate="G$1" pin="2"/>
+<wire x1="73.66" y1="-96.52" x2="76.2" y2="-96.52" width="0.1524" layer="91"/>
+<wire x1="73.66" y1="-104.14" x2="73.66" y2="-96.52" width="0.1524" layer="91"/>
+<junction x="73.66" y="-96.52"/>
 </segment>
 </net>
@@
 <segment>
 <pinref part="IC1" gate="G$1" pin="RD"/>
-<wire x1="25.4" y1="0" x2="30.48" y2="0" width="0.1524" layer="91"/>
-<label x="30.48" y="0" size="1.4224" layer="95" xref="yes"/>
+<wire x1="25.4" y1="0" x2="45.72" y2="0" width="0.1524" layer="91"/>
+<label x="55.88" y="0" size="1.4224" layer="95" xref="yes"/>
+<pinref part="R15" gate="G$1" pin="1"/>
+<wire x1="45.72" y1="0" x2="55.88" y2="0" width="0.1524" layer="91"/>
+<wire x1="45.72" y1="2.54" x2="45.72" y2="0" width="0.1524" layer="91"/>
+<junction x="45.72" y="0"/>
 </segment>
 <segment>
@@
 <segment>
 <pinref part="IC1" gate="G$1" pin="WR"/>
-<wire x1="25.4" y1="-2.54" x2="30.48" y2="-2.54" width="0.1524" layer="91"/>
-<label x="30.48" y="-2.54" size="1.4224" layer="95" xref="yes"/>
-</segment>
-<segment>
+<wire x1="25.4" y1="-2.54" x2="50.8" y2="-2.54" width="0.1524" layer="91"/>
+<label x="55.88" y="-2.54" size="1.4224" layer="95" xref="yes"/>
+<pinref part="R16" gate="G$1" pin="1"/>
+<wire x1="50.8" y1="-2.54" x2="55.88" y2="-2.54" width="0.1524" layer="91"/>
+<wire x1="50.8" y1="2.54" x2="50.8" y2="-2.54" width="0.1524" layer="91"/>
+<junction x="50.8" y="-2.54"/>
+</segment>
+<segment>
