File: hardware/8085_shadow.brd (EAGLE design)
At the start: 167.9 x 122.5 mm, 56 parts, among them IC11 74HCT245DW, IC2 74HCT574N, IC3 74LVC1G04DBV, IC5 74HCT245DW, IC6 74AC273N, IC7 74LVC1G79DBV, IC9 74HCT138N

Commit message: Bug in PCB design fixed
Connections:
- net A14: no longer U$3.27
- net VCC: now also U$3.27
Routing:
- net A14: track 206.5 -> 177.8 mm, vias 6 -> 4
- net VCC: track 695.8 -> 698.3 mm
Changed lines of the file:
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@@
 <wire x1="87.6291" y1="18.923" x2="87.6291" y2="19.0463" width="0.4064" layer="16"/>
 <wire x1="87.6291" y1="19.0463" x2="87.6254" y2="19.05" width="0.4064" layer="16"/>
+<contactref element="U$3" pad="27"/>
+<wire x1="118.745" y1="51.435" x2="118.745" y2="53.975" width="1.016" layer="16"/>
 </signal>
 <signal name="GND">
@@
 <wire x1="155.575" y1="60.325" x2="153.9875" y2="60.325" width="0.4064" layer="16"/>
 <wire x1="153.9875" y1="60.325" x2="140.6525" y2="46.99" width="0.4064" layer="16"/>
-<contactref element="U$3" pad="27"/>
 <wire x1="93.345" y1="51.435" x2="95.25" y2="51.435" width="0.4064" layer="16"/>
 <wire x1="95.25" y1="51.435" x2="96.52" y2="52.705" width="0.4064" layer="16"/>
@@
 <via x="88.9" y="84.455" extent="1-16" drill="0.6" diameter="1.4224" shape="octagon"/>
 <contactref element="IC5" pad="3"/>
-<via x="126.365" y="21.59" extent="1-16" drill="0.6" diameter="1.4224" shape="octagon"/>
 <wire x1="88.9" y1="51.435" x2="93.345" y2="51.435" width="0.4064" layer="16"/>
 <wire x1="101.2825" y1="51.435" x2="99.695" y2="52.705" width="0.4064" layer="16"/>
@@
 <wire x1="80.01" y1="95.885" x2="88.9" y2="86.995" width="0.4064" layer="16"/>
 <wire x1="88.9" y1="86.995" x2="88.9" y2="84.455" width="0.4064" layer="16"/>
-<via x="126.365" y="45.72" extent="1-16" drill="0.6" diameter="1.4224" shape="octagon"/>
-<wire x1="126.365" y1="21.59" x2="126.365" y2="45.72" width="0.4064" layer="1"/>
 <wire x1="130.81" y1="45.72" x2="132.08" y2="46.99" width="0.4064" layer="16"/>
 <wire x1="132.08" y1="46.99" x2="140.6525" y2="46.99" width="0.4064" layer="16"/>
 <contactref element="U$2" pad="1"/>
-<wire x1="115.8875" y1="45.72" x2="126.365" y2="45.72" width="0.4064" layer="16"/>
-<wire x1="126.365" y1="45.72" x2="130.81" y2="45.72" width="0.4064" layer="16"/>
-<wire x1="117.1575" y1="53.975" x2="118.745" y2="53.975" width="0.4064" layer="16"/>
-<wire x1="115.8875" y1="51.435" x2="115.8875" y2="52.705" width="0.4064" layer="16"/>
-<wire x1="115.8875" y1="52.705" x2="117.1575" y2="53.975" width="0.4064" layer="16"/>
+<wire x1="115.8875" y1="45.72" x2="130.81" y2="45.72" width="0.4064" layer="16"/>
 <wire x1="101.2825" y1="51.435" x2="113.665" y2="51.435" width="0.4064" layer="16"/>
 <wire x1="113.665" y1="51.435" x2="115.8875" y2="51.435" width="0.6096" layer="16"/>
@@
 <contactref element="U$3" pad="20"/>
 <via x="123.825" y="70.485" extent="1-16" drill="0.6" diameter="1.4224" shape="octagon"/>
-<via x="123.825" y="21.59" extent="1-16" drill="0.6" diameter="1.4224" shape="octagon"/>
+<via x="123.825" y="24.13" extent="1-16" drill="0.6" diameter="1.4224" shape="octagon"/>
 <wire x1="118.745" y1="71.755" x2="120.65" y2="71.755" width="0.4064" layer="16"/>
 <wire x1="120.65" y1="71.755" x2="121.92" y2="70.485" width="0.4064" layer="16"/>
 <wire x1="121.92" y1="70.485" x2="123.825" y2="70.485" width="0.4064" layer="16"/>
-<wire x1="123.825" y1="21.59" x2="123.825" y2="70.485" width="0.4064" layer="1"/>
+<wire x1="123.825" y1="24.13" x2="123.825" y2="70.485" width="0.4064" layer="1"/>
 <contactref element="IC4" pad="14"/>
-<wire x1="123.825" y1="21.59" x2="123.825" y2="19.3675" width="0.4064" layer="16"/>
+<wire x1="123.825" y1="24.13" x2="123.825" y2="19.3675" width="0.6096" layer="16"/>
 </signal>
 <signal name="OUT_4">
@@
 <via x="111.125" y="21.59" extent="1-16" drill="0.6" diameter="1.4224" shape="octagon"/>
 <contactref element="IC4" pad="19"/>
-<wire x1="111.125" y1="21.59" x2="111.125" y2="19.3675" width="0.4064" layer="16"/>
+<wire x1="111.125" y1="21.59" x2="111.125" y2="19.3675" width="0.6096" layer="16"/>
 </signal>
 <signal name="INTA">
@@
 <wire x1="79.0575" y1="8.5725" x2="103.1875" y2="8.5725" width="0.4064" layer="16"/>
 <wire x1="103.1875" y1="8.5725" x2="104.775" y2="10.16" width="0.4064" layer="16"/>
-<wire x1="104.775" y1="10.16" x2="104.775" y2="15.875" width="0.4064" layer="16"/>
-<wire x1="104.775" y1="15.875" x2="106.045" y2="17.145" width="0.4064" layer="16"/>
-<wire x1="106.045" y1="17.145" x2="106.045" y2="19.3675" width="0.4064" layer="16"/>
+<wire x1="104.775" y1="10.16" x2="104.775" y2="14.605" width="0.4064" layer="16"/>
+<wire x1="104.775" y1="14.605" x2="106.045" y2="15.875" width="0.4064" layer="16"/>
+<wire x1="106.045" y1="15.875" x2="106.045" y2="19.3675" width="0.4064" layer="16"/>
 <wire x1="79.0575" y1="8.5725" x2="64.4525" y2="23.1775" width="0.4064" layer="16"/>
 <wire x1="64.4525" y1="24.765" x2="64.4525" y2="23.1775" width="0.4064" layer="16"/>
@@
 <wire x1="118.745" y1="16.1925" x2="118.745" y2="11.7475" width="0.4064" layer="16"/>
 <wire x1="72.0725" y1="10.795" x2="77.7875" y2="5.08" width="0.4064" layer="16"/>
-<wire x1="77.7875" y1="5.08" x2="113.9825" y2="5.08" width="0.4064" layer="16"/>
-<wire x1="113.9825" y1="5.08" x2="118.745" y2="9.8425" width="0.4064" layer="16"/>
+<wire x1="77.7875" y1="5.08" x2="107.315" y2="5.08" width="0.4064" layer="16"/>
 <wire x1="118.745" y1="9.8425" x2="118.745" y2="11.7475" width="0.4064" layer="16"/>
+<wire x1="107.315" y1="5.08" x2="110.8075" y2="8.5725" width="0.4064" layer="16"/>
+<wire x1="110.8075" y1="8.5725" x2="117.475" y2="8.5725" width="0.4064" layer="16"/>
+<wire x1="117.475" y1="8.5725" x2="118.745" y2="9.8425" width="0.4064" layer="16"/>
 </signal>
 <signal name="IO_M">
@@
 <wire x1="92.075" y1="3.81" x2="135.255" y2="3.81" width="0.4064" layer="16"/>
 <contactref element="IC7" pad="1"/>
-<wire x1="90.2154" y1="17.46" x2="92.075" y2="17.46" width="0.4064" layer="16"/>
+<wire x1="90.2154" y1="17.46" x2="92.075" y2="17.46" width="0.6096" layer="16"/>
 </signal>
 <signal name="LOCAL_PORT_CS">
@@
 <wire x1="106.68" y1="87.63" x2="103.505" y2="87.63" width="0.4064" layer="16"/>
 <contactref element="IC4" pad="22"/>
-<wire x1="103.505" y1="21.9075" x2="103.505" y2="19.3675" width="0.4064" layer="16"/>
+<wire x1="103.505" y1="21.9075" x2="103.505" y2="19.3675" width="0.6096" layer="16"/>
 </signal>
 <signal name="N$3">
@@
 <wire x1="78.74" y1="7.62" x2="60.325" y2="26.035" width="0.4064" layer="16"/>
 <contactref element="IC4" pad="17"/>
-<wire x1="113.665" y1="6.0325" x2="117.475" y2="9.8425" width="0.4064" layer="16"/>
-<wire x1="117.475" y1="9.8425" x2="117.475" y2="16.51" width="0.4064" layer="16"/>
+<wire x1="117.475" y1="10.16" x2="117.475" y2="16.51" width="0.4064" layer="16"/>
 <wire x1="117.475" y1="16.51" x2="116.205" y2="17.78" width="0.4064" layer="16"/>
 <wire x1="116.205" y1="17.78" x2="116.205" y2="19.3675" width="0.4064" layer="16"/>
-<wire x1="113.665" y1="6.0325" x2="90.17" y2="6.0325" width="0.4064" layer="16"/>
+<wire x1="106.9975" y1="6.0325" x2="90.17" y2="6.0325" width="0.4064" layer="16"/>
 <wire x1="90.17" y1="6.0325" x2="88.5825" y2="7.62" width="0.4064" layer="16"/>
 <wire x1="88.5825" y1="7.62" x2="78.74" y2="7.62" width="0.4064" layer="16"/>
+<wire x1="106.9975" y1="6.0325" x2="110.49" y2="9.525" width="0.4064" layer="16"/>
+<wire x1="110.49" y1="9.525" x2="116.84" y2="9.525" width="0.4064" layer="16"/>
+<wire x1="116.84" y1="9.525" x2="117.475" y2="10.16" width="0.4064" layer="16"/>
 </signal>
 <signal name="N$29">
